Commit message: commit

File: description/gazebo_control.xacro (robot description, xacro)
@@ -8,7 +8,14 @@
             <wheel_separation>0.45</wheel_separation>
             <wheel_diameter>0.15</wheel_diameter>
+            <!-- Flippers Information -->
+            <flipper_joint_left>left_flipper_joint</flipper_joint_left>
+            <flipper_joint_right>right_flipper_joint</flipper_joint_right>
+            <flipper_separation>0.65</flipper_separation>
+            <flipper_length>0.4</flipper_length>
             <!-- Limits -->
             <max_wheel_torque>200</max_wheel_torque>
             <max_wheel_acceleration>10.0</max_wheel_acceleration>
+            <max_flipper_torque>50</max_flipper_torque>
+            <max_flipper_angle>1.57</max_flipper_angle>
             <!-- Output -->
             <odometry_frame>odom</odometry_frame>

File: description/robot_core.xacro (robot description, xacro)
@@ -161,24 +161,29 @@
     </gazebo>
     <!-- RIGHT FLIBER WHEEL LINK -->
-    <joint name="right_flibber_wheel_joint" type="fixed">
-        <parent link="base_link" />
+    <joint name="right_flibber_wheel_joint" type="revolute">
+        <parent link="right_font_wheel" />
         <child link="right_flibber_wheel" />
-        <origin xyz="0.6 -0.325 0.08" rpy="0 -${pi/8} 0" />
         <axis xyz="0 1 0" />
-    </joint>
+        <limit lower="0" upper="${pi}" effort="100" velocity="100"/>
+    </joint>
+    <xacro:property name="arm_length" value="0.4" />
+    <xacro:property name="arm_H" value="0.1" />
+    <xacro:property name="arm_W" value="0.1" />
+    <xacro:property name="arm_radius" value="0.15" />
     <link name="right_flibber_wheel">
         <visual>
-            <geometry>
-                <box size="0.4 0.1 0.1" />
-            </geometry>
-            <material name="blue" />
-        </visual>
-        <collision>
-            <geometry>
-                <box size="0.4 0.1 0.1" />
-            </geometry>
-        </collision>
-        <xacro:inertial_cylinder mass="0.1" length="0.4" radius="0.15">
-            <origin xyz="0 0 0" rpy="0 0 0" />
+            <origin xyz="${arm_length/2} 0 0" rpy="0 ${pi} 0" />
+            <geometry>
+                <box size="${arm_length} ${arm_H} ${arm_W}" />
+            </geometry>
+            <material name="blue" />
+        </visual>
+        <collision>
+            <geometry>
+                <box size="${arm_length} ${arm_H} ${arm_W}" />
+            </geometry>
+        </collision>
+        <xacro:inertial_cylinder mass="0.1" length="${arm_length}" radius="${arm_radius}">
+            <origin xyz="${arm_length/2} 0 0" rpy="0 ${pi} 0" />
         </xacro:inertial_cylinder>
     </link>
@@ -189,23 +194,25 @@
     </gazebo>
     <!-- LEFT FLIBBER WHEEL LINK -->
-    <joint name="left_flibber_wheel_joint" type="fixed">
-        <parent link="base_link" />
+    <joint name="left_flibber_wheel_joint" type="revolute">
+        <parent link="left_font_wheel" />
         <child link="left_flibber_wheel" />
-        <origin xyz="0.6 0.325 0.08" rpy="0 -${pi/8} 0" />
+        <origin xyz="${arm_length} 0 0" rpy="0 -${pi} 0" />
         <axis xyz="0 -1 0" />
+        <limit lower="0" upper="${pi}" effort="100" velocity="100"/>
     </joint>
     <link name="left_flibber_wheel">
         <visual>
-            <geometry>
-                <box size="0.4 0.1 0.1" />
-            </geometry>
-            <material name="blue" />
-        </visual>
-        <collision>
-            <geometry>
-                <box size="0.4 0.1 0.1" />
-            </geometry>
-        </collision>
-        <xacro:inertial_cylinder mass="0.1" length="0.4" radius="0.15">
+            <origin xyz="${arm_length/2} 0 0" rpy="0 ${pi} 0" />
+            <geometry>
+                 <box size="${arm_length} ${arm_H} ${arm_W}" />
+            </geometry>
+            <material name="blue" />
+        </visual>
+        <collision>
+            <geometry>
+                 <box size="${arm_length} ${arm_H} ${arm_W}" />
+            </geometry>
+        </collision>
+        <xacro:inertial_cylinder mass="0.1" length="${arm_length}" radius="${arm_radius}">
             <origin xyz="0 0 0" rpy="0 0 0" />
         </xacro:inertial_cylinder>
@@ -217,5 +224,5 @@
     </gazebo>
     <!-- LEFT TRACK-->
-    <joint name="left_track_joint" type="fixed">
+    <!-- <joint name="left_track_joint" type="fixed">
         <parent link="base_link" />
         <child link="left_track_wheel" />
@@ -243,7 +250,7 @@
         <mu1 value="0.001" />
         <mu2 value="0.001" />
-    </gazebo>
+    </gazebo> -->
     <!-- RIGHT TRACK-->
-    <joint name="right_track_joint" type="fixed">
+    <!-- <joint name="right_track_joint" type="fixed">
         <parent link="base_link" />
         <child link="right_track_wheel" />
@@ -271,4 +278,4 @@
         <mu1 value="0.001" />
         <mu2 value="0.001" />
-    </gazebo>
+    </gazebo> -->
 </robot>

Commit message: commit

File: description/gazebo_control.xacro (robot description, xacro)
@@ -9,6 +9,6 @@
             <wheel_diameter>0.15</wheel_diameter>
             <!-- Flippers Information -->
-            <flipper_joint_left>left_flipper_joint</flipper_joint_left>
-            <flipper_joint_right>right_flipper_joint</flipper_joint_right>
+            <flipper_joint_left>left_flibber_wheel_joint</flipper_joint_left>
+            <flipper_joint_right>right_flibber_wheel_joint</flipper_joint_right>
             <flipper_separation>0.65</flipper_separation>
             <flipper_length>0.4</flipper_length>
@@ -24,4 +24,5 @@
             <publish_odom_tf>true</publish_odom_tf>
             <publish_wheel_tf>true</publish_wheel_tf>
+            <publish_flipper_tf>true</publish_flipper_tf>
         </plugin>
     </gazebo>

File: description/robot_core.xacro (robot description, xacro)
@@ -162,67 +162,66 @@
     <!-- RIGHT FLIBER WHEEL LINK -->
     <joint name="right_flibber_wheel_joint" type="revolute">
-        <parent link="right_font_wheel" />
-        <child link="right_flibber_wheel" />
-        <axis xyz="0 1 0" />
-        <limit lower="0" upper="${pi}" effort="100" velocity="100"/>
+        <origin xyz="-0.075 0 0.1" rpy="0 0 0"/>
+        <parent link="right_font_wheel"/>
+        <child link="right_flibber_wheel"/>
+        <axis xyz="0 0 1"/>
+        <limit lower="0" upper="${pi/2}" velocity="100" effort="100"/>
     </joint>
     <xacro:property name="arm_length" value="0.4" />
-    <xacro:property name="arm_H" value="0.1" />
-    <xacro:property name="arm_W" value="0.1" />
-    <xacro:property name="arm_radius" value="0.15" />
+    <xacro:property name="arm_radius" value="0.075" />
     <link name="right_flibber_wheel">
         <visual>
-            <origin xyz="${arm_length/2} 0 0" rpy="0 ${pi} 0" />
-            <geometry>
-                <box size="${arm_length} ${arm_H} ${arm_W}" />
-            </geometry>
-            <material name="blue" />
-        </visual>
-        <collision>
-            <geometry>
-                <box size="${arm_length} ${arm_H} ${arm_W}" />
-            </geometry>
-        </collision>
-        <xacro:inertial_cylinder mass="0.1" length="${arm_length}" radius="${arm_radius}">
-            <origin xyz="${arm_length/2} 0 0" rpy="0 ${pi} 0" />
+            <origin xyz="${arm_length/2} 0 0" rpy="0 ${pi/2} 0"/>
+            <geometry>
+                <cylinder length="${arm_length}" radius="${arm_radius}" />
+            </geometry>
+            <material name="orange" />
+        </visual>
+        <collision>
+            <origin xyz="${arm_length/2} 0 0" rpy="0 ${pi/2} 0"/>
+            <geometry>
+                <cylinder length="${arm_length}" radius="${arm_radius}" />
+            </geometry>
+        </collision>
+        <xacro:inertial_cylinder mass="1.0" length="${arm_length}" radius="${arm_radius}">
+            <origin xyz="${arm_length/2} 0 0" rpy="0 ${pi/2} 0"/>
         </xacro:inertial_cylinder>
     </link>
     <gazebo reference="right_flibber_wheel">
         <material>Gazebo/Black</material>
-        <mu1 value="0.001" />
-        <mu2 value="0.001" />
     </gazebo>
     <!-- LEFT FLIBBER WHEEL LINK -->
-    <joint name="left_flibber_wheel_joint" type="revolute">
-        <parent link="left_font_wheel" />
-        <child link="left_flibber_wheel" />
-        <origin xyz="${arm_length} 0 0" rpy="0 -${pi} 0" />
-        <axis xyz="0 -1 0" />
-        <limit lower="0" upper="${pi}" effort="100" velocity="100"/>
-    </joint>
+   <joint name="left_flibber_wheel_joint" type="revolute">
+        <origin xyz="-0.075 0 0.1" rpy="0 0 0"/>
+        <parent link="left_font_wheel"/>
+        <child link="left_flibber_wheel"/>
+        <axis xyz="0 0 -1"/>
+        <limit lower="0" upper="${pi/2}" velocity="100" effort="100"/>
+    </joint>
+    <xacro:property name="arm_length" value="0.4" />
+    <xacro:property name="arm_radius" value="0.075" />
     <link name="left_flibber_wheel">
         <visual>
-            <origin xyz="${arm_length/2} 0 0" rpy="0 ${pi} 0" />
-            <geometry>
-                 <box size="${arm_length} ${arm_H} ${arm_W}" />
-            </geometry>
-            <material name="blue" />
-        </visual>
-        <collision>
-            <geometry>
-                 <box size="${arm_length} ${arm_H} ${arm_W}" />
-            </geometry>
-        </collision>
-        <xacro:inertial_cylinder mass="0.1" length="${arm_length}" radius="${arm_radius}">
-            <origin xyz="0 0 0" rpy="0 0 0" />
+            <origin xyz="${arm_length/2} 0 0" rpy="0 ${pi/2} 0"/>
+            <geometry>
+                <cylinder length="${arm_length}" radius="${arm_radius}" />
+            </geometry>
+            <material name="orange" />
+        </visual>
+        <collision>
+            <origin xyz="${arm_length/2} 0 0" rpy="0 ${pi/2} 0"/>
+            <geometry>
+                <cylinder length="${arm_length}" radius="${arm_radius}" />
+            </geometry>
+        </collision>
+        <xacro:inertial_cylinder mass="1.0" length="${arm_length}" radius="${arm_radius}">
+            <origin xyz="${arm_length/2} 0 0" rpy="0 ${pi/2} 0"/>
         </xacro:inertial_cylinder>
     </link>
     <gazebo reference="left_flibber_wheel">
         <material>Gazebo/Black</material>
-        <mu1 value="0.001" />
-        <mu2 value="0.001" />
     </gazebo>
     <!-- LEFT TRACK-->
-    <!-- <joint name="left_track_joint" type="fixed">
+    <joint name="left_track_joint" type="fixed">
         <parent link="base_link" />
         <child link="left_track_wheel" />
@@ -250,7 +249,7 @@
         <mu1 value="0.001" />
         <mu2 value="0.001" />
-    </gazebo> -->
+    </gazebo>
     <!-- RIGHT TRACK-->
-    <!-- <joint name="right_track_joint" type="fixed">
+    <joint name="right_track_joint" type="fixed">
         <parent link="base_link" />
         <child link="right_track_wheel" />
@@ -278,4 +277,4 @@
         <mu1 value="0.001" />
         <mu2 value="0.001" />
-    </gazebo> -->
+    </gazebo>
 </robot>
