Commit message: commit

File: description/robot.urdf.xacro (robot description, xacro)
@@ -1,15 +1,16 @@
 <?xml version="1.0"?>
 <robot xmlns:xacro="http://www.ros.org/wiki/xacro"  name="robot">
-    <!-- <xacro:arg name="use_ros2_control" default="true"/>
-    <xacro:arg name="sim_mode" default="false"/> -->
+    <xacro:arg name="use_ros2_control" default="true"/>
+    <xacro:arg name="sim_mode" default="false"/>
     <xacro:include filename="robot_core.xacro" />
-    <!-- <xacro:if value="$(arg use_ros2_control)"> -->
+    <xacro:if value="$(arg use_ros2_control)">
         <xacro:include filename="ros2_control.xacro" />
-    <!-- </xacro:if> -->
-    <!-- <xacro:unless value="$(arg use_ros2_control)"> -->
+    </xacro:if>
+    <xacro:unless value="$(arg use_ros2_control)">
         <xacro:include filename="gazebo_control.xacro" />
-    <!-- </xacro:unless> -->
+    </xacro:unless>
     <xacro:include filename="lidar.xacro" />
     <!-- <xacro:include filename="camera.xacro" /> -->
     <!-- <xacro:include filename="depth_camera.xacro" /> -->
+    <!-- <xacro:include filename="face.xacro" /> -->
 </robot>

File: description/robot_core.urdf (robot description, URDF)
Before this commit: robot hendbot, 15 links, 14 joints
Links:
- link hend_link: mass 43.4880454963273 -> 430.4880454963273

File: description/robot_core.xacro (robot description, xacro)
@@ -35,5 +35,5 @@
         rpy="0 0 0" />
       <mass
-        value="43.4880454963273" />
+        value="430.4880454963273" />
       <inertia
         ixx="0.580105726031867"
@@ -137,6 +137,6 @@
      <gazebo reference="RBW_Link">
         <material>Gazebo/Orange</material>
-        <mu1 value="0.1" />
-        <mu2 value="0.1" />
+        <mu1 value="0.04" />
+        <mu2 value="0.04" />
     </gazebo>
   <link
@@ -201,6 +201,6 @@
       <gazebo reference="LBW_Link">
         <material>Gazebo/Orange</material>
-        <mu1 value="0.1" />
-        <mu2 value="0.1" />
+        <mu1 value="0.04" />
+        <mu2 value="0.04" />
     </gazebo>
   <link
@@ -389,6 +389,6 @@
     <gazebo reference="RFW_Link">
         <material>Gazebo/Orange</material>
-        <mu1 value="0.1" />
-        <mu2 value="0.1" />
+        <mu1 value="0.04" />
+        <mu2 value="0.04" />
     </gazebo>
   <link
@@ -453,6 +453,6 @@
     <gazebo reference="LFW_Link">
         <material>Gazebo/Orange</material>
-        <mu1 value="0.1" />
-        <mu2 value="0.1" />
+        <mu1 value="0.04" />
+        <mu2 value="0.04" />
     </gazebo>
   <link
@@ -519,6 +519,6 @@
     <gazebo reference="RFFW_Link">
         <material>Gazebo/Orange</material>
-        <mu1 value="0.1" />
-        <mu2 value="0.1" />
+        <mu1 value="0.04" />
+        <mu2 value="0.04" />
     </gazebo>
   <link
@@ -643,6 +643,6 @@
     <gazebo reference="RW_Link">
         <material>Gazebo/Orange</material>
-        <mu1 value="0.1" />
-        <mu2 value="0.1" />
+        <mu1 value="0.04" />
+        <mu2 value="0.04" />
     </gazebo>
   <link
@@ -709,6 +709,6 @@
     <gazebo reference="LFFW_Link">
         <material>Gazebo/Orange</material>
-        <mu1 value="0.1" />
-        <mu2 value="0.1" />
+        <mu1 value="0.04" />
+        <mu2 value="0.04" />
     </gazebo>
   <link
@@ -828,6 +828,6 @@
       <gazebo reference="LW_Link">
         <material>Gazebo/Orange</material>
-        <mu1 value="0.1" />
-        <mu2 value="0.1" />
+        <mu1 value="0.04" />
+        <mu2 value="0.04" />
     </gazebo>
 </robot>

File: description/ros2_control.xacro (robot description, xacro)
@@ -1,61 +1,28 @@
 <?xml version="1.0"?>
 <robot xmlns:xacro="http://www.ros.org/wiki/xacro">
-    <xacro:unless value="$(arg sim_mode)">
-        <ros2_control name="RealRobot" type="system">
-            <hardware>
-                <plugin>diffdrive_arduino/DiffDriveArduino</plugin>
-                <param name="left_wheel_name">WLBelt_Joint</param>
-                <param name="right_wheel_name">WRBelt_Joint</param>
-                <param name="loop_rate">30</param>
-                <param name="device">/dev/ttyACM0</param>
-                <param name="baud_rate">57600</param>
-                <param name="timeout">1000</param>
-                <param name="enc_counts_per_rev">80</param>
-            </hardware>
-            <joint name="WLBelt_Joint">
-                <command_interface name="velocity">
-                    <param name="min">-10</param>
-                    <param name="max">10</param>
-                </command_interface>
-                <state_interface name="velocity"/>
-                <state_interface name="position"/>
-            </joint>
-            <joint name="WRBelt_Joint">
-                <command_interface name="velocity">
-                    <param name="min">-10</param>
-                    <param name="max">10</param>
-                </command_interface>
-                <state_interface name="velocity"/>
-                <state_interface name="position"/>
-            </joint>
-        </ros2_control>
-    </xacro:unless>
-    <xacro:if value="$(arg sim_mode)">
-        <ros2_control name="GazeboSystem" type="system">
-            <hardware>
-                <plugin>gazebo_ros2_control/GazeboSystem</plugin>
-            </hardware>
-            <joint name="WLBelt_Joint">
-                <command_interface name="velocity">
-                    <param name="min">-10</param>
-                    <param name="max">10</param>
-                </command_interface>
-                <state_interface name="velocity"/>
-                <state_interface name="position"/>
-            </joint>
-            <joint name="WRBelt_Joint">
-                <command_interface name="velocity">
-                    <param name="min">-10</param>
-                    <param name="max">10</param>
-                </command_interface>
-                <state_interface name="velocity"/>
-                <state_interface name="position"/>
-            </joint>
-        </ros2_control>
-    </xacro:if>
+    <ros2_control name="GazeboSystem" type="system">
+        <hardware>
+            <plugin>gazebo_ros2_control/GazeboSystem</plugin>
+        </hardware>
+        <joint name="WLBelt_Joint">
+            <command_interface name="velocity">
+                <param name="min">-10</param>
+                <param name="max">10</param>
+            </command_interface>
+            <state_interface name="velocity"/>
+            <state_interface name="position"/>
+        </joint>
+        <joint name="WRBelt_Joint">
+            <command_interface name="velocity">
+                <param name="min">-10</param>
+                <param name="max">10</param>
+            </command_interface>
+            <state_interface name="velocity"/>
+            <state_interface name="position"/>
+        </joint>
+    </ros2_control>
     <gazebo>
         <plugin name="gazebo_ros2_control" filename="libgazebo_ros2_control.so">
             <parameters>$(find hendbot)/config/my_controllers.yaml</parameters>
-            <parameters>$(find hendbot)/config/gaz_ros2_ctl_use_sim.yaml</parameters>
         </plugin>
     </gazebo>
